Commit message: RB1 spawned in warehouse

File: my_rb1_description/urdf/materials.xacro (robot description, xacro)
@@ -2,5 +2,8 @@
 <robot name="my_rb1_robot" xmlns:xacro="http://www.ros.org/wiki/xacro" >
 <material name="silver">
-  <color rgba="0.700 0.700 0.700 1.000"/>
+  <color rgba="1.0 1.0 1.0 0.5"/>
+</material>
+<material name="black">
+  <color rgba="1.0 1.0 1.0 0.5"/>
 </material>
 </robot>

File: my_rb1_description/urdf/my_rb1_robot.xacro (robot description, xacro)
@@ -15,5 +15,5 @@
       <mesh filename="package://my_rb1_description/meshes/base_link.stl" scale="0.001 0.001 0.001"/>
     </geometry>
-    <material name="silver"/>
+    <material name="black"/>
   </visual>
   <collision>
